Commit message: YAWJOINT修正

File: double_arm_tnk_description/urdf/MANI_ARM.urdf.xacro (robot description, xacro)
@@ -155,5 +155,5 @@
       <mass value="22.9404" />
       <origin xyz="-0.169575 0 0.000436442" rpy="0 -0 0" />
-      <inertia ixx="0.0917743" ixy="0" ixz="-0.000933033" iyy="0.193104" iyz="0" izz="0, 0.221433" />
+      <inertia ixx="0.0917743" ixy="0" ixz="-0.000933033" iyy="0.193104" iyz="0" izz="0.221433" />
     </inertial>
   </link>
