Commit message: 慣性特性を修正

File: double_arm_tnk_description/urdf/BASE.urdf.xacro (robot description, xacro)
@@ -179,7 +179,7 @@
     </collision>
     <inertial>
-      <mass value="1e-06" />
-      <origin xyz="0 0 0" rpy="0 -0 0" />
-      <inertia ixx="1.0" ixy="0.0" ixz="0.0" iyy="1.0" iyz="0.0" izz="1.0" />
+      <mass value="445" />
+      <origin xyz="2.61167950E-02 -2.48536360E-01 7.38255770E-05" rpy="0 -0 0" />
+      <inertia ixx="1.17125210E+02" ixy="9.30859190E-01" ixz="7.71323470E-03" iyy="2.13308730E+02" iyz="-4.07759970E-03" izz="1.08880120E+02" />
     </inertial>
   </link>

File: double_arm_tnk_description/urdf/MANI_ARM.urdf.xacro (robot description, xacro)
@@ -57,7 +57,7 @@
     </collision>
     <inertial>
-      <mass value="1e-06" />
-      <origin xyz="0 0 0" rpy="0 -0 0" />
-      <inertia ixx="1.0" ixy="0.0" ixz="0.0" iyy="1.0" iyz="0.0" izz="1.0" />
+      <mass value="535.84647" />
+      <origin xyz="8.14422630E-02 1.99598060E-01 2.71745980E-02" rpy="0 -0 0" />
+      <inertia ixx="7.97084620E+01" ixy="-8.47185310E+00" ixz="1.11603580E+00" iyy="1.00038320E+02" iyz="5.51320690E+00" izz="6.17888570E+01" />
     </inertial>
   </link>
@@ -77,7 +77,7 @@
     </collision>
     <inertial>
-      <mass value="1e-06" />
-      <origin xyz="0 0 0" rpy="0 -0 0" />
-      <inertia ixx="1.0" ixy="0.0" ixz="0.0" iyy="1.0" iyz="0.0" izz="1.0" />
+      <mass value="1.3380749e+01" />
+      <origin xyz="-6.7856551e-2 9.6877149e-3 0.0000000e+00" rpy="0 -0 0" />
+      <inertia ixx="5.9129940e-02" ixy="-3.7243340e-03" ixz="0.0000000e+00" iyy="3.5238822e-02" iyz="0.0000000e+00" izz="7.3441120e-02" />
     </inertial>
   </link>
@@ -133,7 +133,7 @@
     </collision>
     <inertial>
-      <mass value="1e-06" />
-      <origin xyz="0 0 0" rpy="0 -0 0" />
-      <inertia ixx="1.0" ixy="0.0" ixz="0.0" iyy="1.0" iyz="0.0" izz="1.0" />
+      <mass value="2.3976610e+01" />
+      <origin xyz="-4.7393726e-2 -3.4379664e-2 0.0000000e+00" rpy="0 -0 0" />
+      <inertia ixx="1.5009182e-1" ixy="6.9121654e-2" ixz="0.0000000e+00" iyy="1.8822635e-1" iyz="0.0000000e+00" izz="2.3426912e-1" />
     </inertial>
   </link>
@@ -153,7 +153,7 @@
     </collision>
     <inertial>
-      <mass value="1e-06" />
-      <origin xyz="0 0 0" rpy="0 -0 0" />
-      <inertia ixx="1.0" ixy="0.0" ixz="0.0" iyy="1.0" iyz="0.0" izz="1.0" />
+      <mass value="22.9404" />
+      <origin xyz="-0.169575 0 0.000436442" rpy="0 -0 0" />
+      <inertia ixx="0.0917743" ixy="0" ixz="-0.000933033" iyy="0.193104" iyz="0" izz="0, 0.221433" />
     </inertial>
   </link>
@@ -173,7 +173,7 @@
     </collision>
     <inertial>
-      <mass value="1e-06" />
-      <origin xyz="0 0 0" rpy="0 -0 0" />
-      <inertia ixx="1.0" ixy="0.0" ixz="0.0" iyy="1.0" iyz="0.0" izz="1.0" />
+      <mass value="4.08874" />
+      <origin xyz="-0.106437 0 0" rpy="0 -0 0" />
+      <inertia ixx="0.00678026" ixy="0" ixz="0" iyy="0.0266742" iyz="0" izz="0.0241877" />
     </inertial>
   </link>
@@ -187,7 +187,7 @@
     </visual>
     <inertial>
-      <mass value="1e-06" />
-      <origin xyz="0 0 0" rpy="0 -0 0" />
-      <inertia ixx="1.0" ixy="0.0" ixz="0.0" iyy="1.0" iyz="0.0" izz="1.0" />
+      <mass value="0.887605" />
+      <origin xyz="0.0512686 0 0" rpy="0 -0 0" />
+      <inertia ixx="0.000237569" ixy="0" ixz="0" iyy="0.00159781" iyz="0" izz="0.00159822" />
     </inertial>
   </link>

File: double_arm_tnk_description/urdf/TOHOKU_ARM.urdf.xacro (robot description, xacro)
@@ -39,7 +39,7 @@
     </collision>
     <inertial>
-      <mass value="1e-06" />
-      <origin xyz="0 0 0" rpy="0 -0 0" />
-      <inertia ixx="1.0" ixy="0.0" ixz="0.0" iyy="1.0" iyz="0.0" izz="1.0" />
+      <mass value="455.45935" />
+      <origin xyz="7.35035370E-02 1.06590700E-01 1.61371410E-02" rpy="0 -0 0" />
+      <inertia ixx="4.19870890E+01" ixy="1.70520040E+00" ixz="-6.24433200E+00" iyy="9.66620960E+01" iyz="-6.61440150E-01" izz="6.14020130E+01" />
     </inertial>
   </link>
@@ -59,7 +59,7 @@
     </collision>
     <inertial>
-      <mass value="1e-06" />
-      <origin xyz="0 0 0" rpy="0 -0 0" />
-      <inertia ixx="1.0" ixy="0.0" ixz="0.0" iyy="1.0" iyz="0.0" izz="1.0" />
+      <mass value="27.099865985502" />
+      <origin xyz="-6.78385281318872e-002 1.77765761382185e-002 -6.67318029447292e-003" rpy="0 -0 0" />
+      <inertia ixx="0.328996567191697" ixy="5.52858323486756e-003" ixz="5.74693929208142e-003" iyy="0.160727640206049" iyz="-1.33419251009407e-002" izz="0.319147626929996" />
     </inertial>
   </link>
@@ -115,7 +115,7 @@
     </collision>
     <inertial>
-      <mass value="1e-06" />
-      <origin xyz="0 0 0" rpy="0 -0 0" />
-      <inertia ixx="1.0" ixy="0.0" ixz="0.0" iyy="1.0" iyz="0.0" izz="1.0" />
+      <mass value="2.1377092e+01" />
+      <origin xyz="-1.2434069e-1 -6.6741207e-3 0.0000000e+00" rpy="0 -0 0" />
+      <inertia ixx="2.4528689e-1" ixy="7.1716531e-3" ixz="0.0000000e+00" iyy="1.8144181e-1" iyz="0.0000000e+00" izz="2.1758796e-1" />
     </inertial>
   </link>
@@ -135,7 +135,7 @@
     </collision>
     <inertial>
-      <mass value="1e-06" />
-      <origin xyz="0 0 0" rpy="0 -0 0" />
-      <inertia ixx="1.0" ixy="0.0" ixz="0.0" iyy="1.0" iyz="0.0" izz="1.0" />
+      <mass value="5.6820888e+01" />
+      <origin xyz="-1.0832237e-1  0.0000000e+00  0.0000000e+00" rpy="0 -0 0" />
+      <inertia ixx="7.8278692e-1" ixy="0.0000000e+00" ixz="0.0000000e+00" iyy="7.0832807e-1" iyz="0.0000000e+00" izz="1.1161951e-1" />
     </inertial>
   </link>
@@ -155,7 +155,7 @@
     </collision>
     <inertial>
-      <mass value="1e-06" />
-      <origin xyz="0 0 0" rpy="0 -0 0" />
-      <inertia ixx="1.0" ixy="0.0" ixz="0.0" iyy="1.0" iyz="0.0" izz="1.0" />
+      <mass value="9.3058947e+00" />
+      <origin xyz="-1.9052236e-1  1.1160593e-1 -7.5632562e-04" rpy="0 -0 0" />
+      <inertia ixx="3.0276157e-2" ixy="1.1688229e-2" ixz="1.2268932e-3" iyy="1.5080350e-2" iyz="-7.1011455e-4" izz="1.8011625e-1" />
     </inertial>
   </link>
@@ -175,7 +175,7 @@
     </collision>
     <inertial>
-      <mass value="1e-06" />
-      <origin xyz="0 0 0" rpy="0 -0 0" />
-      <inertia ixx="1.0" ixy="0.0" ixz="0.0" iyy="1.0" iyz="0.0" izz="1.0" />
+      <mass value="9.3058947e+00" />
+      <origin xyz="-1.9052236e-1  1.1160593e-1 -7.5632562e-04" rpy="0 -0 0" />
+      <inertia ixx="3.0276157e-2" ixy="1.1688229e-2" ixz="1.2268932e-3" iyy="1.5080350e-2" iyz="-7.1011455e-4" izz="1.8011625e-1" />
     </inertial>
   </link>
