Commit message: UFRAMEとMFRAMEだけの慣性特性をオリジナルに戻す．

File: double_arm_tnk_description/urdf/DoubleArmV7A-TNK.urdf (robot description, URDF)
Before this commit: robot DoubleArmV7-TNK, 36 links, 35 joints
Links:
- link MFRAME: mass 455.45935E-3 -> 455.45935
- link UFRAME: mass 535.84647E-3 -> 535.84647

File: double_arm_tnk_description/urdf/MANI_ARM.urdf.xacro (robot description, xacro)
@@ -57,7 +57,7 @@
     </collision>
     <inertial>
-      <mass value="535.84647E-3" />
+      <mass value="535.84647" />
       <origin xyz="8.14422630E-02 1.99598060E-01 2.71745980E-02" rpy="0 -0 0" />
-      <inertia ixx="7.97084620E-4" ixy="-8.47185310E-5" ixz="1.11603580E-5" iyy="1.00038320E-3" iyz="5.51320690E-5" izz="6.17888570E-4" />
+      <inertia ixx="7.97084620E+01" ixy="-8.47185310E+00" ixz="1.11603580E+00" iyy="1.00038320E+02" iyz="5.51320690E+00" izz="6.17888570E+01" />
     </inertial>
   </link>

File: double_arm_tnk_description/urdf/TOHOKU_ARM.urdf.xacro (robot description, xacro)
@@ -39,7 +39,7 @@
     </collision>
     <inertial>
-      <mass value="455.45935E-3" />
+      <mass value="455.45935" />
       <origin xyz="7.35035370E-02 1.06590700E-01 1.61371410E-02" rpy="0 -0 0" />
-      <inertia ixx="4.19870890E-4" ixy="1.70520040E-5" ixz="-6.24433200E-5" iyy="9.66620960E-4" iyz="-6.61440150E-6" izz="6.14020130E-4" />
+      <inertia ixx="4.19870890E+01" ixy="1.70520040E+00" ixz="-6.24433200E+00" iyy="9.66620960E+01" iyz="-6.61440150E-01" izz="6.14020130E+01" />
     </inertial>
   </link>
